File: _autosave-discipline-pcb.kicad_pcb (KiCad board)
At the start: 4 copper layers, 304.9 x 122.8 mm, 169 parts, among them SW1 KEYSW, SW10 KEYSW, SW11 KEYSW, SW12 KEYSW, SW13 KEYSW, SW14 KEYSW, SW15 KEYSW, SW16 KEYSW, SW17 KEYSW, SW18 KEYSW, SW19 KEYSW, SW2 KEYSW, SW20 KEYSW, SW21 KEYSW, SW22 KEYSW, SW23 KEYSW, SW24 KEYSW, SW25 KEYSW, SW26 KEYSW, SW27 KEYSW, SW28 KEYSW, SW29 KEYSW, SW3 KEYSW, SW30 KEYSW, SW31 KEYSW, SW32 KEYSW, SW33 KEYSW, SW34 KEYSW, SW35 KEYSW, SW36 KEYSW, SW37 KEYSW, SW38 KEYSW, SW39 KEYSW, SW4 KEYSW, SW40 KEYSW, SW41 KEYSW, SW42 KEYSW, SW43 KEYSW, SW44 KEYSW, SW45 KEYSW, SW46 KEYSW, SW47 KEYSW, SW48 KEYSW, SW49 KEYSW, SW5 KEYSW, SW50 KEYSW, SW51 KEYSW, SW52 KEYSW, SW53 KEYSW, SW54 KEYSW, SW55 KEYSW, SW56 KEYSW, SW57 KEYSW, SW58 KEYSW, SW59 KEYSW, SW6 KEYSW, SW60 KEYSW, SW61 KEYSW, SW62 KEYSW, SW63 KEYSW, SW64 KEYSW, SW65 KEYSW, SW66 KEYSW, SW67 KEYSW, SW68 KEYSW, SW69 KEYSW, SW7 KEYSW, SW70 KEYSW, SW71 KEYSW, SW72 KEYSW, SW73 KEYSW, SW74 KEYSW, SW75 KEYSW, SW76 KEYSW, SW77 KEYSW, SW78 KEYSW, SW79 SW_SPST, SW8 KEYSW, SW9 KEYSW, U1 SuperMini nRF52840

Commit message: Versão base com nice
Parts:
- removed SW70, SW73, SW74: KEYSW, cftkb:SW_Cherry_MX1A_1.50u_PCBNOSCREEN
- removed SW76: KEYSW, cftkb:SW_Cherry_MX1A_ISOEnter_PCB_ReversedStabilizer
Connections:
- net /VBAT_RAW renamed V_BAT
- J_BAT1 pad 2: /GND_BAT -> GND
- U1 pad 14: unconnected-(U1-GND-Pad14) -> GND
- U1 pad 28: /GND_BAT -> GND
- U1 pad 3: unconnected-(U1-GND-Pad3) -> GND
- U1 pad 4: unconnected-(U1-GND-Pad4) -> GND
Routing:
- net col10: track 186.7 -> 172.5 mm
- net /GND_BAT: track 13.4 -> 0.00 mm
- net col9: track 192.0 -> 187.2 mm
- net Net-(D63-A): track 279.4 -> 274.6 mm
- added copper zone on F.Cu, net GND
- removed copper zone on F.Cu, net (none)
