File: _autosave-discipline-pcb.kicad_pcb (KiCad board)
At the start: 4 copper layers, 304.9 x 122.8 mm, 169 parts, among them SW1 KEYSW, SW10 KEYSW, SW11 KEYSW, SW12 KEYSW, SW13 KEYSW, SW14 KEYSW, SW15 KEYSW, SW16 KEYSW, SW17 KEYSW, SW18 KEYSW, SW19 KEYSW, SW2 KEYSW, SW20 KEYSW, SW21 KEYSW, SW22 KEYSW, SW23 KEYSW, SW24 KEYSW, SW25 KEYSW, SW26 KEYSW, SW27 KEYSW, SW28 KEYSW, SW29 KEYSW, SW3 KEYSW, SW30 KEYSW, SW31 KEYSW, SW32 KEYSW, SW33 KEYSW, SW34 KEYSW, SW35 KEYSW, SW36 KEYSW, SW37 KEYSW, SW38 KEYSW, SW39 KEYSW, SW4 KEYSW, SW40 KEYSW, SW41 KEYSW, SW42 KEYSW, SW43 KEYSW, SW44 KEYSW, SW45 KEYSW, SW46 KEYSW, SW47 KEYSW, SW48 KEYSW, SW49 KEYSW, SW5 KEYSW, SW50 KEYSW, SW51 KEYSW, SW52 KEYSW, SW53 KEYSW, SW54 KEYSW, SW55 KEYSW, SW56 KEYSW, SW57 KEYSW, SW58 KEYSW, SW59 KEYSW, SW6 KEYSW, SW60 KEYSW, SW61 KEYSW, SW62 KEYSW, SW63 KEYSW, SW64 KEYSW, SW65 KEYSW, SW66 KEYSW, SW67 KEYSW, SW68 KEYSW, SW69 KEYSW, SW7 KEYSW, SW70 KEYSW, SW71 KEYSW, SW72 KEYSW, SW73 KEYSW, SW74 KEYSW, SW75 KEYSW, SW76 KEYSW, SW77 KEYSW, SW78 KEYSW, SW79 SW_SPST, SW8 KEYSW, SW9 KEYSW, U1 SuperMini nRF52840

Commit message: Removing keys for the ISO layout
Parts:
- removed D71: ~, cftkb:D_DO-35_SOD27_P5.08mm_Horizontal
- removed SW69, SW78: KEYSW, cftkb:SW_Cherry_MX1A_1.25u_PCBNOSCREEN
- removed SW70, SW71, SW73, SW74: KEYSW, cftkb:SW_Cherry_MX1A_1.50u_PCBNOSCREEN
- removed SW72, SW75, SW77: KEYSW, cftkb:SW_Cherry_MX1A_1.00u_PCB-NOSCREEN
- removed SW76: KEYSW, cftkb:SW_Cherry_MX1A_ISOEnter_PCB_ReversedStabilizer
Routing:
- net row3: track 438.8 -> 297.0 mm, vias 4 -> 1
- net Net-(D61-A): track 425.1 -> 408.5 mm
- net Net-(D71-A): track 15.0 -> 0.00 mm
- net col10: track 186.5 -> 172.2 mm
- net col2: track 337.0 -> 324.4 mm
- net col13: track 117.2 -> 105.3 mm
- net Net-(D43-A): track 153.6 -> 142.4 mm
- net col0: track 378.4 -> 368.1 mm
- net Net-(D29-A): track 127.9 -> 118.4 mm
- net Net-(D45-A): track 85.1 -> 75.6 mm
- net col6: track 242.5 -> 236.8 mm
- net col9: track 192.0 -> 187.2 mm
- net Net-(D63-A): track 279.4 -> 274.6 mm
- net Net-(D31-A): track 69.7 -> 65.0 mm
- net Net-(D59-A): track 462.2 -> 459.8 mm
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Other:
- board text removed: "1.25U ISO"
- board text removed: "1.5U"
- board text removed: "1U ISO"
- board text removed: "ISO"
- board text removed: "ISO ENTER"
- board text removed: "STEPPED"
