File: discipline-pcb.kicad_pcb (KiCad board)
At the start: 4 copper layers, 304.9 x 122.8 mm, 169 parts, among them SW1 KEYSW, SW10 KEYSW, SW11 KEYSW, SW12 KEYSW, SW13 KEYSW, SW14 KEYSW, SW15 KEYSW, SW16 KEYSW, SW17 KEYSW, SW18 KEYSW, SW19 KEYSW, SW2 KEYSW, SW20 KEYSW, SW21 KEYSW, SW22 KEYSW, SW23 KEYSW, SW24 KEYSW, SW25 KEYSW, SW26 KEYSW, SW27 KEYSW, SW28 KEYSW, SW29 KEYSW, SW3 KEYSW, SW30 KEYSW, SW31 KEYSW, SW32 KEYSW, SW33 KEYSW, SW34 KEYSW, SW35 KEYSW, SW36 KEYSW, SW37 KEYSW, SW38 KEYSW, SW39 KEYSW, SW4 KEYSW, SW40 KEYSW, SW41 KEYSW, SW42 KEYSW, SW43 KEYSW, SW44 KEYSW, SW45 KEYSW, SW46 KEYSW, SW47 KEYSW, SW48 KEYSW, SW49 KEYSW, SW5 KEYSW, SW50 KEYSW, SW51 KEYSW, SW52 KEYSW, SW53 KEYSW, SW54 KEYSW, SW55 KEYSW, SW56 KEYSW, SW57 KEYSW, SW58 KEYSW, SW59 KEYSW, SW6 KEYSW, SW60 KEYSW, SW61 KEYSW, SW62 KEYSW, SW63 KEYSW, SW64 KEYSW, SW65 KEYSW, SW66 KEYSW, SW67 KEYSW, SW68 KEYSW, SW69 KEYSW, SW7 KEYSW, SW70 KEYSW, SW71 KEYSW, SW72 KEYSW, SW73 KEYSW, SW74 KEYSW, SW75 KEYSW, SW76 KEYSW, SW77 KEYSW, SW78 KEYSW, SW79 SW_SPST, SW8 KEYSW, SW9 KEYSW, U1 SuperMini nRF52840

Commit message: Finishing JLCPCB support and implementing decoupling capacitors
Parts:
- removed D71: ~, cftkb:D_DO-35_SOD27_P5.08mm_Horizontal
- removed G*** (x2): LOGO, logos:TOPY 4MM MASK
- removed G***: LOGO, logos:rev1-1_16mm_mask
- removed G***: LOGO, logos:coseyfannitutti_16mm
- removed G***: LOGO, logos:DISCIPLINE_SMALL_MASK
- removed ST72: 7U, cftkb:MX-7U-Stabilizer
- removed SW69, SW78: KEYSW, cftkb:SW_Cherry_MX1A_1.25u_PCBNOSCREEN
- removed SW70, SW71, SW73, SW74: KEYSW, cftkb:SW_Cherry_MX1A_1.50u_PCBNOSCREEN
- removed SW72, SW75, SW77: KEYSW, cftkb:SW_Cherry_MX1A_1.00u_PCB-NOSCREEN
- removed SW76: KEYSW, cftkb:SW_Cherry_MX1A_ISOEnter_PCB_ReversedStabilizer
- added C1: 100nF, Capacitor_THT:C_Rect_L11.5mm_W5.2mm_P10.00mm_MKT, F.Cu at (337.5, 82.2)
- added C2: 10µF, Capacitor_THT:C_Disc_D4.7mm_W2.5mm_P5.00mm, F.Cu at (350.5, 83.0)
- moved SW79 13.9 mm to (354.2, 68.2), turned to 0 degrees
Connections:
- U1 pad 16: unconnected-(U1-3V3-Pad16) -> Net-(U1-3V3)
Routing:
- net row3: track 438.8 -> 297.0 mm, vias 4 -> 0
- net Net-(D61-A): track 425.1 -> 408.5 mm
- net Net-(D71-A): track 15.0 -> 0.00 mm
- net col13: track 117.2 -> 102.8 mm
- net col10: track 186.5 -> 172.2 mm
- net col2: track 337.0 -> 324.3 mm
- net col0: track 378.4 -> 367.9 mm
- net /VBAT_SW: track 3.53 -> 13.8 mm
- net Net-(D29-A): track 127.9 -> 118.4 mm
- net Net-(D45-A): track 85.1 -> 76.0 mm
- net Net-(D57-A): track 152.2 -> 159.5 mm
- net col6: track 242.5 -> 236.8 mm
- net V_BAT: track 19.2 -> 14.3 mm
- net col9: track 192.0 -> 187.2 mm
- net Net-(D63-A): track 279.4 -> 274.6 mm
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Other:
- board text added: "(void*()())&((int()(void))0xDEADBEEF); int i=i+1; (int)0xCAFE = 0; (long long)(char)(void*)0; p = (int*)malloc(42); int i = 0;"
- board text added: "1"
- board text added: "I know this hole should not be this way"
- board text added: "Rev 1.0 - 2025"
- board text added: "char* s = {dblquote}foo{dblquote}; while(*s++); // string length? (void)(*(volatile int*)0x4B1D); 0xFEEDFACE; for(i=0; i<10; --i); free(malloc(10)); // bluetooth conn"
- board text added: "free(p); p = 1; goto hell; float f = (float)i / 0.0f; (unsigned char)(int)(void*)0; 0[arr]++; int x = y = z = 0; (int)(((float)&i));"
- board text added: "int x; return &x; // returning address of local variable. (void*)*((int*)0); 0xBADF00D; (char)0xFF << 8; (int)(1.0f / 0.0f); // Inf. //Mem leak"
- board text added: "void* void* void* void* void* void* void* void* void* void* void* void* void* void* void* void* void* void* void* void*"
- board text added: "void* void* void* void* void* void* void* void* void* void* void* void* void* void* void* void* void* void* void* void* void* void* void* void*"
- board text removed: "1.25U"
- board text removed: "1.25U ISO"
- board text removed: "1.5U"
- board text removed: "1U"
- board text removed: "1U ISO"
- board text removed: "2.25U ANSI"
- board text removed: "ANSI ENTER"
- board text removed: "ISO"
- board text removed: "ISO ENTER"
- board text removed: "STANDARD"
- board text removed: "STEPPED"

Commit message: Adding GND plane to back layer and rerouting
Parts:
- moved J_BAT1 4.45 mm to (336.1, 69.4)
Connections:
- U1 pad 11: col3 -> col4
- U1 pad 12: col4 -> col3
Routing:
- net Net-(D43-A): track 149.0 -> 159.7 mm
- net Net-(D57-A): track 159.5 -> 169.6 mm
- net row0: track 299.0 -> 290.6 mm
- net row3: track 297.0 -> 289.1 mm
- net col3: track 280.8 -> 275.4 mm
- net V_BAT: track 14.3 -> 18.7 mm
- net Net-(D50-A): track 114.4 -> 110.4 mm
- net Net-(D51-A): track 119.9 -> 116.4 mm
- net Net-(D37-A): track 90.0 -> 86.5 mm
- net Net-(D22-A): track 68.6 -> 65.1 mm
- net Net-(D7-A): track 46.2 -> 43.0 mm
- net Net-(D52-A): track 125.9 -> 122.7 mm
- net Net-(D8-A): track 52.3 -> 49.3 mm
- net Net-(D23-A): track 74.5 -> 71.5 mm
- net Net-(D38-A): track 95.6 -> 92.8 mm
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- added copper zone on B.Cu, net GND
- removed copper zone on B.Cu, net (none)
Other:
- outline, holes or cut-outs redrawn
- board text removed: "(void*()())&((int()(void))0xDEADBEEF); int i=i+1; (int)0xCAFE = 0; (long long)(char)(void*)0; p = (int*)malloc(42); int i = 0;"
- board text removed: "I know this hole should not be this way"
- board text removed: "char* s = {dblquote}foo{dblquote}; while(*s++); // string length? (void)(*(volatile int*)0x4B1D); 0xFEEDFACE; for(i=0; i<10; --i); free(malloc(10)); // bluetooth conn"
- board text removed: "free(p); p = 1; goto hell; float f = (float)i / 0.0f; (unsigned char)(int)(void*)0; 0[arr]++; int x = y = z = 0; (int)(((float)&i));"
- board text removed: "int x; return &x; // returning address of local variable. (void*)*((int*)0); 0xBADF00D; (char)0xFF << 8; (int)(1.0f / 0.0f); // Inf. //Mem leak"
- board text removed: "void* void* void* void* void* void* void* void* void* void* void* void* void* void* void* void* void* void* void* void*"
- board text removed: "void* void* void* void* void* void* void* void* void* void* void* void* void* void* void* void* void* void* void* void* void* void* void* void*"

Commit message: Removing files that are not usefull
Other:
- copper layers 4 -> 2
- board text removed: "1"
