File: voidPointer-pcb.kicad_sch (KiCad schematic)
At the start: 152 parts, among them SW1 KEYSW, SW10 KEYSW, SW11 KEYSW, SW12 KEYSW, SW13 KEYSW, SW14 KEYSW, SW15 KEYSW, SW16 KEYSW, SW17 KEYSW, SW18 KEYSW, SW19 KEYSW, SW2 KEYSW, SW20 KEYSW, SW21 KEYSW, SW22 KEYSW, SW23 KEYSW, SW24 KEYSW, SW25 KEYSW, SW26 KEYSW, SW27 KEYSW, SW28 KEYSW, SW29 KEYSW, SW3 KEYSW, SW30 KEYSW, SW31 KEYSW, SW32 KEYSW, SW33 KEYSW, SW34 KEYSW, SW35 KEYSW, SW36 KEYSW, SW37 KEYSW, SW38 KEYSW, SW39 KEYSW, SW4 KEYSW, SW40 KEYSW, SW41 KEYSW, SW42 KEYSW, SW43 KEYSW, SW44 KEYSW, SW45 KEYSW, SW46 KEYSW, SW47 KEYSW, SW48 KEYSW, SW49 KEYSW, SW5 KEYSW, SW50 KEYSW, SW51 KEYSW, SW52 KEYSW, SW53 KEYSW, SW54 KEYSW, SW55 KEYSW, SW56 KEYSW, SW57 KEYSW, SW58 KEYSW, SW59 KEYSW, SW6 KEYSW, SW60 KEYSW, SW61 KEYSW, SW62 KEYSW, SW63 KEYSW, SW64 KEYSW, SW65 KEYSW, SW66 KEYSW, SW67 KEYSW, SW68 KEYSW, SW69 KEYSW, SW7 KEYSW, SW70 KEYSW, SW71 KEYSW, SW72 KEYSW, SW73 KEYSW, SW74 KEYSW, SW75 KEYSW, SW76 KEYSW, SW77 KEYSW, SW78 KEYSW, SW79 SW_SPST, SW8 KEYSW, SW9 KEYSW, U1 SuperMini nRF52840

Commit message: Renaming project revision and title
Other:
- note added: "1.0"
- note added: "void* // 65% keyboard with only through hole components adapted from Discipline"
- note removed: "1.1"
- note removed: "void* // 65% keyboard with only through hole components"
Changed lines of the file:
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@@
 	(generator_version "9.0")
 	(paper "A3")
-	(text "1.1"
+	(text "1.0"
 		(exclude_from_sim no)
 		(at 394.97 280.67 0)
@@
 		)
 	)
-	(text "void* // 65% keyboard with only through hole components"
+	(text "void* // 65% keyboard with only through hole components adapted from Discipline"
 		(exclude_from_sim no)
 		(at 302.26 255.27 0)
