File: plate/discipline-pcb.kicad_pcb (KiCad board)
At the start: 2 copper layers, 305.8 x 96.2 mm, 3 parts

Commit message: Removing files that are not usefull
Parts:
- removed G***: LOGO, logos:coseyfannitutti_16mm
- removed G***: LOGO, logos:DISCIPLINE_SMALL_COPPER
- removed G***: LOGO, logos:DISCIPLINE_SMALL_MASK
Other:
- net class Default removed
